Commit message: fix: update Revomate joint3/5 URDF parameters

File: revoarm_system/urdf/revoarm_bimanual_revo2.urdf (robot description, URDF)
Before this commit: robot revoarm_bimanual, 66 links, 65 joints
Joints:
- joint revoarm_left_joint3: limit lower=-3.6652 upper=0.5236 effort=27 velocity=1.745 -> lower=-2.0 upper=2.0 effort=27 velocity=1.745
- joint revoarm_left_joint5: limit lower=-3.1444 upper=0.9044 effort=7 velocity=6.98 -> lower=-3.1444 upper=0.500 effort=7 velocity=6.98

Commit message: fix: update Revomate URDF parameters right-arm

File: revoarm_system/urdf/revoarm_bimanual_revo2.urdf (robot description, URDF)
Before this commit: robot revoarm_bimanual, 66 links, 65 joints
Joints:
- joint revoarm_right_joint3: limit lower=-3.6652 upper=0.5236 effort=27 velocity=1.745 -> lower=-2.0 upper=2.0 effort=27 velocity=1.745
- joint revoarm_right_joint5: limit lower=-3.1444 upper=0.9044 effort=7 velocity=6.98 -> lower=-3.1444 upper=0.500 effort=7 velocity=6.98
