Commit message: feat : change revotron/revo3 offset

File: revotron_system/urdf/revotron_bimanual_revo3.urdf (robot description, URDF)
Before this commit: robot revotron_bimanual, 78 links, 77 joints
Joints:
- joint left_connector_mount: origin xyz=0 -0.095 0 rpy=0.0 0.785 3.14 -> xyz=0 -0.095 0 rpy=0.0 2.355 3.14
- joint right_connector_mount: origin xyz=0 -0.095 0 rpy=0.0 0.785 3.14 -> xyz=0 -0.095 0 rpy=0.0 -0.785 3.14

File: revotron_system/urdf/revotron_single_left_revo3.urdf (robot description, URDF)
Before this commit: robot revotron_single, 40 links, 39 joints
Joints:
- joint left_connector_mount: origin xyz=0 -0.095 0 rpy=0.0 0.785 3.14 -> xyz=0 -0.095 0 rpy=0.0 2.355 3.14

File: revotron_system/urdf/revotron_single_right_revo3.urdf (robot description, URDF)
Before this commit: robot revotron_single, 40 links, 39 joints
Joints:
- joint right_connector_mount: origin xyz=0 -0.095 0 rpy=0.0 0.785 3.14 -> xyz=0 -0.095 0 rpy=0.0 -0.785 3.14

Commit message: feat: change revotron bimanual initial position

File: revotron_system/urdf/revotron_bimanual_revo3.urdf (robot description, URDF)
Before this commit: robot revotron_bimanual, 78 links, 77 joints
Joints:
- joint base_to_left_arm: origin xyz=0 0.08 1.270 rpy=-1.57 0 0 -> xyz=0 0.08 1.270 rpy=-1.57 -1.57 0
- joint base_to_right_arm: origin xyz=0 -0.08 1.270 rpy=1.57 0 0 -> xyz=0 -0.08 1.270 rpy=1.57 -1.57 0
