Commit message: Add Revotron camera coordinate frames and wrist cameras
Add the head OAK camera and left/right wrist camera meshes, with updated
camera coordinate frames, mounting transforms, and inertial properties.
Update Revotron wrist connectors and regenerate the corresponding MJCF
and USD models. Include the current URDF formatting and refreshed USD
assets for Revo2, Revo3, and RevoArm.

Validation: link/body and movable joint names are consistent across all
30 URDF/USD/MJCF model sets, accounting for generated USD root joints
and omitted MJCF fixed joints/world bodies. Changed XML files parse
successfully and all referenced meshes exist.

File: revotron_system/urdf/revotron_bimanual_revo3.urdf (robot description, URDF)
Before this commit: robot revotron_bimanual, 142 links, 141 joints
Links:
- removed link head_camera_link
- added link head_oak_link, mass 0.10003; collision mesh filename=../meshes/arm/collision/Head_Oak_Link.STL; visual mesh filename=../meshes/arm/visual/Head_Oak_Link.STL
- link head_Link: mass 1.345 -> 1.245
- link left_connector_link: mass 0.113854752828569 -> 0.25057
- link left_wrist_camera_frame: mass None -> 0.049871; geometry collision mesh filename=../meshes/arm/collision/left_wrist_camera_link.STL; visual mesh filename=../meshes/arm/visual/left_wrist_camera_link.STL
- link right_connector_link: mass 0.11385419870144 -> 0.25057
- link right_wrist_camera_frame: mass None -> 0.049871; geometry collision mesh filename=../meshes/arm/collision/right_wrist_camera_link.STL; visual mesh filename=../meshes/arm/visual/right_wrist_camera_link.STL
Joints:
- removed joint head_camera_joint
- added joint head_oak_joint: type fixed, parent head_Link, child head_oak_link, origin xyz=0.085038 0 0.092986 rpy=0 0.78539 0
- joint left_connector_mount: origin xyz=0 -0.095 0 rpy=-1.57 1.57 0.0 -> xyz=0 -0.10695 0 rpy=-1.5707963267948966 0 3.141592653589793
- joint left_connector_tip_joint: origin xyz=0 0.00 -0.018 rpy=3.14 0.0 1.57 -> xyz=0 0 0 rpy=0 0 0
- joint left_wrist_camera_joint: origin xyz=0.0528 0.07508 -0.0225 rpy=-0.34906585 0.34906585 0 -> xyz=0.072095 0.035586 0.030977 rpy=0.51561 0 0
- joint right_connector_mount: origin xyz=0 -0.095 0 rpy=-1.57 -1.57 0.0 -> xyz=0 -0.10695 0 rpy=1.5707963267948966 0 0
- joint right_connector_tip_joint: origin xyz=0 0.00 -0.018 rpy=3.14 0.0 1.57 -> xyz=0 0 0 rpy=0 0 0
- joint right_wrist_camera_joint: origin xyz=-0.0528 0.07508 -0.0225 rpy=-0.34906585 -0.34906585 0 -> xyz=0.035478911816555 0.0724666383278956 0.0307759368724696 rpy=-0.51560789253163 0 1.5707963267949

File: revotron_system/urdf/revotron_bimanual_revo3_mx_touch.urdf (robot description, URDF)
Before this commit: robot revotron_bimanual, 636 links, 635 joints
Links:
- removed link head_camera_link
- added link head_oak_link, mass 0.10003; collision mesh filename=../meshes/arm/collision/Head_Oak_Link.STL; visual mesh filename=../meshes/arm/visual/Head_Oak_Link.STL
- link head_Link: mass 1.345 -> 1.245
- link left_connector_link: mass 0.113854752828569 -> 0.25057
- link left_wrist_camera_frame: mass None -> 0.049871; geometry collision mesh filename=../meshes/arm/collision/left_wrist_camera_link.STL; visual mesh filename=../meshes/arm/visual/left_wrist_camera_link.STL
- link right_connector_link: mass 0.11385419870144 -> 0.25057
- link right_wrist_camera_frame: mass None -> 0.049871; geometry collision mesh filename=../meshes/arm/collision/right_wrist_camera_link.STL; visual mesh filename=../meshes/arm/visual/right_wrist_camera_link.STL
Joints:
- removed joint head_camera_joint
- added joint head_oak_joint: type fixed, parent head_Link, child head_oak_link, origin xyz=0.085038 0 0.092986 rpy=0 0.78539 0
- joint left_connector_mount: origin xyz=0 -0.095 0 rpy=-1.57 1.57 0.0 -> xyz=0 -0.10695 0 rpy=-1.5707963267948966 0 3.141592653589793
- joint left_connector_tip_joint: origin xyz=0 0.00 -0.018 rpy=3.14 0.0 1.57 -> xyz=0 0 0 rpy=0 0 0
- joint left_wrist_camera_joint: origin xyz=0.0528 0.07508 -0.0225 rpy=-0.34906585 0.34906585 0 -> xyz=0.072095 0.035586 0.030977 rpy=0.51561 0 0
- joint right_connector_mount: origin xyz=0 -0.095 0 rpy=-1.57 -1.57 0.0 -> xyz=0 -0.10695 0 rpy=1.5707963267948966 0 0
- joint right_connector_tip_joint: origin xyz=0 0.00 -0.018 rpy=3.14 0.0 1.57 -> xyz=0 0 0 rpy=0 0 0
- joint right_wrist_camera_joint: origin xyz=-0.0528 0.07508 -0.0225 rpy=-0.34906585 -0.34906585 0 -> xyz=0.035478911816555 0.0724666383278956 0.0307759368724696 rpy=-0.51560789253163 0 1.5707963267949

File: revotron_system/urdf/revotron_single_left_revo3.urdf (robot description, URDF)
Before this commit: robot revotron_single, 70 links, 69 joints
Links:
- link left_connector_link: mass 0.113854752828569 -> 0.25057
- link left_wrist_camera_frame: mass None -> 0.049871; geometry collision mesh filename=../meshes/arm/collision/left_wrist_camera_link.STL; visual mesh filename=../meshes/arm/visual/left_wrist_camera_link.STL
Joints:
- joint left_connector_mount: origin xyz=0 -0.095 0 rpy=-1.57 3.14 0.0 -> xyz=0 -0.10695 0 rpy=1.5707963267948966 -1.5707963267948966 0
- joint left_connector_tip_joint: origin xyz=0 0.00 -0.018 rpy=3.14 0.0 1.57 -> xyz=0 0 0 rpy=0 0 0
- joint left_wrist_camera_joint: origin xyz=0.0528 0.07508 -0.0225 rpy=-0.34906585 0.34906585 0 -> xyz=0.072095 0.035586 0.030977 rpy=0.51561 0 0

File: revotron_system/urdf/revotron_single_left_revo3_mx_touch.urdf (robot description, URDF)
Before this commit: robot revotron_single, 317 links, 316 joints
Links:
- link left_connector_link: mass 0.113854752828569 -> 0.25057
- link left_wrist_camera_frame: mass None -> 0.049871; geometry collision mesh filename=../meshes/arm/collision/left_wrist_camera_link.STL; visual mesh filename=../meshes/arm/visual/left_wrist_camera_link.STL
Joints:
- joint left_connector_mount: origin xyz=0 -0.095 0 rpy=-1.57 3.14 0.0 -> xyz=0 -0.10695 0 rpy=1.5707963267948966 -1.5707963267948966 0
- joint left_connector_tip_joint: origin xyz=0 0.00 -0.018 rpy=3.14 0.0 1.57 -> xyz=0 0 0 rpy=0 0 0
- joint left_wrist_camera_joint: origin xyz=0.0528 0.07508 -0.0225 rpy=-0.34906585 0.34906585 0 -> xyz=0.072095 0.035586 0.030977 rpy=0.51561 0 0

File: revotron_system/urdf/revotron_single_right_revo3.urdf (robot description, URDF)
Before this commit: robot revotron_single, 70 links, 69 joints
Links:
- link right_connector_link: mass 0.11385419870144 -> 0.25057
- link right_wrist_camera_frame: mass None -> 0.049871; geometry collision mesh filename=../meshes/arm/collision/right_wrist_camera_link.STL; visual mesh filename=../meshes/arm/visual/right_wrist_camera_link.STL
Joints:
- joint right_connector_mount: origin xyz=0 -0.095 0 rpy=-1.57 3.14 0.0 -> xyz=0 -0.10695 0 rpy=1.5707963267948966 -1.5707963267948966 0
- joint right_connector_tip_joint: origin xyz=0 0.00 -0.018 rpy=3.14 0.0 1.57 -> xyz=0 0 0 rpy=0 0 0
- joint right_wrist_camera_joint: origin xyz=-0.0528 0.07508 -0.0225 rpy=-0.34906585 -0.34906585 0 -> xyz=0.035478911816555 0.0724666383278956 0.0307759368724696 rpy=-0.51560789253163 0 1.5707963267949

File: revotron_system/urdf/revotron_single_right_revo3_mx_touch.urdf (robot description, URDF)
Before this commit: robot revotron_single, 317 links, 316 joints
Links:
- link right_connector_link: mass 0.11385419870144 -> 0.25057
- link right_wrist_camera_frame: mass None -> 0.049871; geometry collision mesh filename=../meshes/arm/collision/right_wrist_camera_link.STL; visual mesh filename=../meshes/arm/visual/right_wrist_camera_link.STL
Joints:
- joint right_connector_mount: origin xyz=0 -0.095 0 rpy=-1.57 3.14 0.0 -> xyz=0 -0.10695 0 rpy=1.5707963267948966 -1.5707963267948966 0
- joint right_connector_tip_joint: origin xyz=0 0.00 -0.018 rpy=3.14 0.0 1.57 -> xyz=0 0 0 rpy=0 0 0
- joint right_wrist_camera_joint: origin xyz=-0.0528 0.07508 -0.0225 rpy=-0.34906585 -0.34906585 0 -> xyz=0.035478911816555 0.0724666383278956 0.0307759368724696 rpy=-0.51560789253163 0 1.5707963267949

Commit message: Release v2026.10.05 with default Revotron appearance
Regenerate robot exports with preserved visual materials and v4 USD physics settings. Add Revotron appearance assets and previews, publish oversized bimanual USD assets through Git LFS, and document the release and validation.

File: revotron_system/urdf/revotron_bimanual_revo3.urdf (robot description, URDF)
Before this commit: robot revotron_bimanual, 142 links, 141 joints
Links:
- link base_link: geometry collision mesh filename=../meshes/body/collision/base_link.STL; visual mesh filename=../meshes/body/visual/appearance/base_link__tron_433c_appro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
- link head_Link: geometry collision mesh filename=../meshes/arm/collision/neck_pitch_Link.STL; visual mesh filename=../meshes/body/visual/appearance/head_Link__tron_433c_appro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
- link waist_Link: geometry collision mesh filename=../meshes/arm/collision/waist_pitch_Link.STL; visual mesh filename=../meshes/body/visual/appearance/waist_Link__tron_cool_gray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

File: revotron_system/urdf/revotron_bimanual_revo3_mx_touch.urdf (robot description, URDF)
Before this commit: robot revotron_bimanual, 636 links, 635 joints
Links:
- link base_link: geometry collision mesh filename=../meshes/body/collision/base_link.STL; visual mesh filename=../meshes/body/visual/appearance/base_link__tron_433c_appro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
- link head_Link: geometry collision mesh filename=../meshes/arm/collision/neck_pitch_Link.STL; visual mesh filename=../meshes/body/visual/appearance/head_Link__tron_433c_appro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
- link waist_Link: geometry collision mesh filename=../meshes/arm/collision/waist_pitch_Link.STL; visual mesh filename=../meshes/body/visual/appearance/waist_Link__tron_cool_gray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
