Commit message: Update Revo3 hand collision geometry across robot models
Add trimmed thumb CMR hulls and backtrimmed palm collision meshes for
both Revo3 hands. Regenerate the Revo3, RevoArm, and Revotron URDF,
MJCF, and USD assets, and refresh the Revo2 USD assets.

Validation: all 30 packaged URDFs parse and resolve mesh paths; 22 Revo3
hand instances in MJCF and USD each contain 32 CMR collision meshes
and one trimmed palm collider. Simulation self-collision behavior still
requires validation.

File: revo3_system/urdf/revo3_left.urdf (robot description, URDF)
Before this commit: robot revo3_single, 58 links, 57 joints
Links:
- link left_plam_link: geometry collision mesh filename=../meshes/hands/collision/left/left_plam_backtrim_v2.obj; visual mesh filename=../meshes/hands/visual/left/left_plam_link__revo3_aluminum.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
- link left_thumb_CMR_link: geometry collision mesh filename=../meshes/hands/collision/left/cmr_v4_00.obj; collision mesh filename=../meshes/hands/collision/left/cmr_v4_01.obj

File: revo3_system/urdf/revo3_left_mx_touch.urdf (robot description, URDF)
Before this commit: robot revo3_single, 305 links, 304 joints
Links:
- link left_plam_link: geometry collision mesh filename=../meshes/hands/collision/left/left_plam_backtrim_v2.obj; visual mesh filename=../meshes/hands/visual/left/left_plam_link__revo3_aluminum.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
- link left_thumb_CMR_link: geometry collision mesh filename=../meshes/hands/collision/left/cmr_v4_00.obj; collision mesh filename=../meshes/hands/collision/left/cmr_v4_01.obj

File: revo3_system/urdf/revo3_right.urdf (robot description, URDF)
Before this commit: robot revo3_single, 58 links, 57 joints
Links:
- link right_plam_link: geometry collision mesh filename=../meshes/hands/collision/right/right_plam_backtrim_v2.obj; visual mesh filename=../meshes/hands/visual/right/right_plam_link__revo3_aluminu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
- link right_thumb_CMR_link: geometry collision mesh filename=../meshes/hands/collision/right/cmr_v4_00.obj; collision mesh filename=../meshes/hands/collision/right/cmr_v4_01.obj

File: revo3_system/urdf/revo3_right_mx_touch.urdf (robot description, URDF)
Before this commit: robot revo3_single, 305 links, 304 joints
Links:
- link right_plam_link: geometry collision mesh filename=../meshes/hands/collision/right/right_plam_backtrim_v2.obj; visual mesh filename=../meshes/hands/visual/right/right_plam_link__revo3_aluminu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
- link right_thumb_CMR_link: geometry collision mesh filename=../meshes/hands/collision/right/cmr_v4_00.obj; collision mesh filename=../meshes/hands/collision/right/cmr_v4_01.obj

File: revoarm_system/urdf/revoarm_bimanual_revo3.urdf (robot description, URDF)
Before this commit: robot revoarm_bimanual, 136 links, 135 joints
Links:
- link left_plam_link: geometry collision mesh filename=../meshes/hands/collision/left/left_plam_backtrim_v2.obj; visual mesh filename=../meshes/hands/visual/left/left_plam_link__revo3_aluminum.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
- link left_thumb_CMR_link: geometry collision mesh filename=../meshes/hands/collision/left/cmr_v4_00.obj; collision mesh filename=../meshes/hands/collision/left/cmr_v4_01.obj
- link right_plam_link: geometry collision mesh filename=../meshes/hands/collision/right/right_plam_backtrim_v2.obj; visual mesh filename=../meshes/hands/visual/right/right_plam_link__revo3_aluminu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
- link right_thumb_CMR_link: geometry collision mesh filename=../meshes/hands/collision/right/cmr_v4_00.obj; collision mesh filename=../meshes/hands/collision/right/cmr_v4_01.obj

File: revoarm_system/urdf/revoarm_bimanual_revo3_mx_touch.urdf (robot description, URDF)
Before this commit: robot revoarm_bimanual, 630 links, 629 joints
Links:
- link left_plam_link: geometry collision mesh filename=../meshes/hands/collision/left/left_plam_backtrim_v2.obj; visual mesh filename=../meshes/hands/visual/left/left_plam_link__revo3_aluminum.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
- link left_thumb_CMR_link: geometry collision mesh filename=../meshes/hands/collision/left/cmr_v4_00.obj; collision mesh filename=../meshes/hands/collision/left/cmr_v4_01.obj
- link right_plam_link: geometry collision mesh filename=../meshes/hands/collision/right/right_plam_backtrim_v2.obj; visual mesh filename=../meshes/hands/visual/right/right_plam_link__revo3_aluminu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
- link right_thumb_CMR_link: geometry collision mesh filename=../meshes/hands/collision/right/cmr_v4_00.obj; collision mesh filename=../meshes/hands/collision/right/cmr_v4_01.obj

File: revoarm_system/urdf/revoarm_single_left_revo3.urdf (robot description, URDF)
Before this commit: robot revoarm_single, 68 links, 67 joints
Links:
- link left_plam_link: geometry collision mesh filename=../meshes/hands/collision/left/left_plam_backtrim_v2.obj; visual mesh filename=../meshes/hands/visual/left/left_plam_link__revo3_aluminum.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
- link left_thumb_CMR_link: geometry collision mesh filename=../meshes/hands/collision/left/cmr_v4_00.obj; collision mesh filename=../meshes/hands/collision/left/cmr_v4_01.obj

File: revoarm_system/urdf/revoarm_single_left_revo3_mx_touch.urdf (robot description, URDF)
Before this commit: robot revoarm_single, 315 links, 314 joints
Links:
- link left_plam_link: geometry collision mesh filename=../meshes/hands/collision/left/left_plam_backtrim_v2.obj; visual mesh filename=../meshes/hands/visual/left/left_plam_link__revo3_aluminum.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
- link left_thumb_CMR_link: geometry collision mesh filename=../meshes/hands/collision/left/cmr_v4_00.obj; collision mesh filename=../meshes/hands/collision/left/cmr_v4_01.obj

File: revoarm_system/urdf/revoarm_single_right_revo3.urdf (robot description, URDF)
Before this commit: robot revoarm_single, 68 links, 67 joints
Links:
- link right_plam_link: geometry collision mesh filename=../meshes/hands/collision/right/right_plam_backtrim_v2.obj; visual mesh filename=../meshes/hands/visual/right/right_plam_link__revo3_aluminu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
- link right_thumb_CMR_link: geometry collision mesh filename=../meshes/hands/collision/right/cmr_v4_00.obj; collision mesh filename=../meshes/hands/collision/right/cmr_v4_01.obj

File: revoarm_system/urdf/revoarm_single_right_revo3_mx_touch.urdf (robot description, URDF)
Before this commit: robot revoarm_single, 315 links, 314 joints
Links:
- link right_plam_link: geometry collision mesh filename=../meshes/hands/collision/right/right_plam_backtrim_v2.obj; visual mesh filename=../meshes/hands/visual/right/right_plam_link__revo3_aluminu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
- link right_thumb_CMR_link: geometry collision mesh filename=../meshes/hands/collision/right/cmr_v4_00.obj; collision mesh filename=../meshes/hands/collision/right/cmr_v4_01.obj

File: revotron_system/urdf/revotron_bimanual_revo3.urdf (robot description, URDF)
Before this commit: robot revotron_bimanual, 142 links, 141 joints
Links:
- link left_plam_link: geometry collision mesh filename=../meshes/hands/collision/left/left_plam_backtrim_v2.obj; visual mesh filename=../meshes/hands/visual/left/left_plam_link__revo3_aluminum.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
- link left_thumb_CMR_link: geometry collision mesh filename=../meshes/hands/collision/left/cmr_v4_00.obj; collision mesh filename=../meshes/hands/collision/left/cmr_v4_01.obj
- link right_plam_link: geometry collision mesh filename=../meshes/hands/collision/right/right_plam_backtrim_v2.obj; visual mesh filename=../meshes/hands/visual/right/right_plam_link__revo3_aluminu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
- link right_thumb_CMR_link: geometry collision mesh filename=../meshes/hands/collision/right/cmr_v4_00.obj; collision mesh filename=../meshes/hands/collision/right/cmr_v4_01.obj
Joints:
- joint right_connector_mount: origin xyz=0 -0.10695 0 rpy=1.5707963267948966 0 0 -> xyz=0 -0.10695 0 rpy=1.5707963267948966 1.5707963267948966 0
- joint right_connector_tip_joint: origin xyz=0 0 0 rpy=0 0 0 -> xyz=0 0 0 rpy=0 0 1.5707963267948966

File: revotron_system/urdf/revotron_bimanual_revo3_mx_touch.urdf (robot description, URDF)
Before this commit: robot revotron_bimanual, 636 links, 635 joints
Links:
- link left_plam_link: geometry collision mesh filename=../meshes/hands/collision/left/left_plam_backtrim_v2.obj; visual mesh filename=../meshes/hands/visual/left/left_plam_link__revo3_aluminum.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
- link left_thumb_CMR_link: geometry collision mesh filename=../meshes/hands/collision/left/cmr_v4_00.obj; collision mesh filename=../meshes/hands/collision/left/cmr_v4_01.obj
- link right_plam_link: geometry collision mesh filename=../meshes/hands/collision/right/right_plam_backtrim_v2.obj; visual mesh filename=../meshes/hands/visual/right/right_plam_link__revo3_aluminu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
- link right_thumb_CMR_link: geometry collision mesh filename=../meshes/hands/collision/right/cmr_v4_00.obj; collision mesh filename=../meshes/hands/collision/right/cmr_v4_01.obj
Joints:
- joint right_connector_mount: origin xyz=0 -0.10695 0 rpy=1.5707963267948966 0 0 -> xyz=0 -0.10695 0 rpy=1.5707963267948966 1.5707963267948966 0
- joint right_connector_tip_joint: origin xyz=0 0 0 rpy=0 0 0 -> xyz=0 0 0 rpy=0 0 1.5707963267948966

File: revotron_system/urdf/revotron_single_left_revo3.urdf (robot description, URDF)
Before this commit: robot revotron_single, 70 links, 69 joints
Links:
- link left_plam_link: geometry collision mesh filename=../meshes/hands/collision/left/left_plam_backtrim_v2.obj; visual mesh filename=../meshes/hands/visual/left/left_plam_link__revo3_aluminum.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
- link left_thumb_CMR_link: geometry collision mesh filename=../meshes/hands/collision/left/cmr_v4_00.obj; collision mesh filename=../meshes/hands/collision/left/cmr_v4_01.obj

File: revotron_system/urdf/revotron_single_left_revo3_mx_touch.urdf (robot description, URDF)
Before this commit: robot revotron_single, 317 links, 316 joints
Links:
- link left_plam_link: geometry collision mesh filename=../meshes/hands/collision/left/left_plam_backtrim_v2.obj; visual mesh filename=../meshes/hands/visual/left/left_plam_link__revo3_aluminum.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
- link left_thumb_CMR_link: geometry collision mesh filename=../meshes/hands/collision/left/cmr_v4_00.obj; collision mesh filename=../meshes/hands/collision/left/cmr_v4_01.obj

File: revotron_system/urdf/revotron_single_right_revo3.urdf (robot description, URDF)
Before this commit: robot revotron_single, 70 links, 69 joints
Links:
- link right_plam_link: geometry collision mesh filename=../meshes/hands/collision/right/right_plam_backtrim_v2.obj; visual mesh filename=../meshes/hands/visual/right/right_plam_link__revo3_aluminu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
- link right_thumb_CMR_link: geometry collision mesh filename=../meshes/hands/collision/right/cmr_v4_00.obj; collision mesh filename=../meshes/hands/collision/right/cmr_v4_01.obj
Joints:
- joint right_connector_mount: origin xyz=0 -0.10695 0 rpy=1.5707963267948966 -1.5707963267948966 0 -> xyz=0 -0.10695 0 rpy=1.5707963267948966 0 0
- joint right_connector_tip_joint: origin xyz=0 0 0 rpy=0 0 0 -> xyz=0 0 0 rpy=0 0 1.5707963267948966

File: revotron_system/urdf/revotron_single_right_revo3_mx_touch.urdf (robot description, URDF)
Before this commit: robot revotron_single, 317 links, 316 joints
Links:
- link right_plam_link: geometry collision mesh filename=../meshes/hands/collision/right/right_plam_backtrim_v2.obj; visual mesh filename=../meshes/hands/visual/right/right_plam_link__revo3_aluminu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
- link right_thumb_CMR_link: geometry collision mesh filename=../meshes/hands/collision/right/cmr_v4_00.obj; collision mesh filename=../meshes/hands/collision/right/cmr_v4_01.obj
Joints:
- joint right_connector_mount: origin xyz=0 -0.10695 0 rpy=1.5707963267948966 -1.5707963267948966 0 -> xyz=0 -0.10695 0 rpy=1.5707963267948966 0 0
- joint right_connector_tip_joint: origin xyz=0 0 0 rpy=0 0 0 -> xyz=0 0 0 rpy=0 0 1.5707963267948966

Commit message: Release 20261009: improve Revo3 appearance

File: revo3_system/urdf/revo3_left.urdf (robot description, URDF)
Before this commit: robot revo3_single, 58 links, 57 joints
Links:
- link left_plam_led_link: geometry collision mesh filename=../meshes/hands/collision/left/left_plam_led_link.STL; visual mesh filename=../meshes/hands/visual/left/left_plam_led_link.dae

File: revo3_system/urdf/revo3_left_mx_touch.urdf (robot description, URDF)
Before this commit: robot revo3_single, 305 links, 304 joints
Links:
- link left_plam_led_link: geometry collision mesh filename=../meshes/hands/collision/left/left_plam_led_link.STL; visual mesh filename=../meshes/hands/visual/left/left_plam_led_link.dae

File: revo3_system/urdf/revo3_right.urdf (robot description, URDF)
Before this commit: robot revo3_single, 58 links, 57 joints
Links:
- link right_plam_led_link: geometry collision mesh filename=../meshes/hands/collision/right/right_plam_led_link.STL; visual mesh filename=../meshes/hands/visual/right/right_plam_led_link.dae

File: revo3_system/urdf/revo3_right_mx_touch.urdf (robot description, URDF)
Before this commit: robot revo3_single, 305 links, 304 joints
Links:
- link right_plam_led_link: geometry collision mesh filename=../meshes/hands/collision/right/right_plam_led_link.STL; visual mesh filename=../meshes/hands/visual/right/right_plam_led_link.dae

File: revoarm_system/urdf/revoarm_bimanual_revo3.urdf (robot description, URDF)
Before this commit: robot revoarm_bimanual, 136 links, 135 joints
Links:
- link left_plam_led_link: geometry collision mesh filename=../meshes/hands/collision/left/left_plam_led_link.STL; visual mesh filename=../meshes/hands/visual/left/left_plam_led_link.dae
- link right_plam_led_link: geometry collision mesh filename=../meshes/hands/collision/right/right_plam_led_link.STL; visual mesh filename=../meshes/hands/visual/right/right_plam_led_link.dae

File: revoarm_system/urdf/revoarm_bimanual_revo3_mx_touch.urdf (robot description, URDF)
Before this commit: robot revoarm_bimanual, 630 links, 629 joints
Links:
- link left_plam_led_link: geometry collision mesh filename=../meshes/hands/collision/left/left_plam_led_link.STL; visual mesh filename=../meshes/hands/visual/left/left_plam_led_link.dae
- link right_plam_led_link: geometry collision mesh filename=../meshes/hands/collision/right/right_plam_led_link.STL; visual mesh filename=../meshes/hands/visual/right/right_plam_led_link.dae

File: revoarm_system/urdf/revoarm_single_left_revo3.urdf (robot description, URDF)
Before this commit: robot revoarm_single, 68 links, 67 joints
Links:
- link left_plam_led_link: geometry collision mesh filename=../meshes/hands/collision/left/left_plam_led_link.STL; visual mesh filename=../meshes/hands/visual/left/left_plam_led_link.dae

File: revoarm_system/urdf/revoarm_single_left_revo3_mx_touch.urdf (robot description, URDF)
Before this commit: robot revoarm_single, 315 links, 314 joints
Links:
- link left_plam_led_link: geometry collision mesh filename=../meshes/hands/collision/left/left_plam_led_link.STL; visual mesh filename=../meshes/hands/visual/left/left_plam_led_link.dae

File: revoarm_system/urdf/revoarm_single_right_revo3.urdf (robot description, URDF)
Before this commit: robot revoarm_single, 68 links, 67 joints
Links:
- link right_plam_led_link: geometry collision mesh filename=../meshes/hands/collision/right/right_plam_led_link.STL; visual mesh filename=../meshes/hands/visual/right/right_plam_led_link.dae

File: revoarm_system/urdf/revoarm_single_right_revo3_mx_touch.urdf (robot description, URDF)
Before this commit: robot revoarm_single, 315 links, 314 joints
Links:
- link right_plam_led_link: geometry collision mesh filename=../meshes/hands/collision/right/right_plam_led_link.STL; visual mesh filename=../meshes/hands/visual/right/right_plam_led_link.dae

File: revotron_system/urdf/revotron_bimanual_revo3.urdf (robot description, URDF)
Before this commit: robot revotron_bimanual, 142 links, 141 joints
Links:
- link left_plam_led_link: geometry collision mesh filename=../meshes/hands/collision/left/left_plam_led_link.STL; visual mesh filename=../meshes/hands/visual/left/left_plam_led_link.dae
- link right_plam_led_link: geometry collision mesh filename=../meshes/hands/collision/right/right_plam_led_link.STL; visual mesh filename=../meshes/hands/visual/right/right_plam_led_link.dae

File: revotron_system/urdf/revotron_bimanual_revo3_mx_touch.urdf (robot description, URDF)
Before this commit: robot revotron_bimanual, 636 links, 635 joints
Links:
- link left_plam_led_link: geometry collision mesh filename=../meshes/hands/collision/left/left_plam_led_link.STL; visual mesh filename=../meshes/hands/visual/left/left_plam_led_link.dae
- link right_plam_led_link: geometry collision mesh filename=../meshes/hands/collision/right/right_plam_led_link.STL; visual mesh filename=../meshes/hands/visual/right/right_plam_led_link.dae

File: revotron_system/urdf/revotron_single_left_revo3.urdf (robot description, URDF)
Before this commit: robot revotron_single, 70 links, 69 joints
Links:
- link left_plam_led_link: geometry collision mesh filename=../meshes/hands/collision/left/left_plam_led_link.STL; visual mesh filename=../meshes/hands/visual/left/left_plam_led_link.dae

File: revotron_system/urdf/revotron_single_left_revo3_mx_touch.urdf (robot description, URDF)
Before this commit: robot revotron_single, 317 links, 316 joints
Links:
- link left_plam_led_link: geometry collision mesh filename=../meshes/hands/collision/left/left_plam_led_link.STL; visual mesh filename=../meshes/hands/visual/left/left_plam_led_link.dae

File: revotron_system/urdf/revotron_single_right_revo3.urdf (robot description, URDF)
Before this commit: robot revotron_single, 70 links, 69 joints
Links:
- link right_plam_led_link: geometry collision mesh filename=../meshes/hands/collision/right/right_plam_led_link.STL; visual mesh filename=../meshes/hands/visual/right/right_plam_led_link.dae

File: revotron_system/urdf/revotron_single_right_revo3_mx_touch.urdf (robot description, URDF)
Before this commit: robot revotron_single, 317 links, 316 joints
Links:
- link right_plam_led_link: geometry collision mesh filename=../meshes/hands/collision/right/right_plam_led_link.STL; visual mesh filename=../meshes/hands/visual/right/right_plam_led_link.dae
